Commit message: remove not used sensors from service robot and add jointpub

File: workspace/src/controller_launch/models/service_robot/plugins.xacro (robot description, xacro)
@@ -12,5 +12,5 @@
                 <pose>0 0 0 0 0 0</pose>
                 <always_on>true</always_on>
-                <visualize>false</visualize>
+                <visualize>true</visualize>
                 <update_rate>5</update_rate>
                 <ray>
@@ -21,6 +21,6 @@
                                  whole rotation, part of which is then cut off -->
                             <resolution>1</resolution>
-                            <min_angle>${min_angle}</min_angle>
-                            <max_angle>${max_angle}</max_angle>
+                            <min_angle>1.571</min_angle>
+                            <max_angle>4.712</max_angle>
                         </horizontal>
                     </scan>
@@ -49,13 +49,13 @@
     <xacro:lidar_plugin
         prefix="lidar_base_front"
-        topic="/lidar/base/front/scan"
-        min_angle="${-1.0*pi}"
-        max_angle="${1.0*pi}"/>
+        topic="scan"
+        min_angle="-1.396263"
+        max_angle="1.396263"/>
         <!-- [-180°;180°] -->
-    <xacro:lidar_plugin
+    <!-- <xacro:lidar_plugin
         prefix="lidar_base_rear"
         topic="/lidar/base/rear/scan"
         min_angle="${-115.0/180*pi}"
-        max_angle="${115.0/180*pi}"/>
+        max_angle="${115.0/180*pi}"/> -->
         <!-- [-115°;115°] -->
     <!-- <joint name="base_joint" type="fixed">
@@ -180,9 +180,9 @@
         </gazebo>
     </xacro:macro>
-    <xacro:marker_camera link="camera_link" topic="camera" fov_horizontal="1.3962634" fov_vertical="1.0471975" width="1200" height="900" rate="5.0"/>
-    <xacro:marker_camera link="camera_top_front_link" topic="camera/top/front" fov_horizontal="1.3962634" fov_vertical="1.0471975" width="1200" height="900" rate="5.0"/>
+    <!-- <xacro:marker_camera link="camera_link" topic="camera" fov_horizontal="1.3962634" fov_vertical="1.0471975" width="1200" height="900" rate="5.0"/> -->
+    <!-- <xacro:marker_camera link="camera_top_front_link" topic="camera/top/front" fov_horizontal="1.3962634" fov_vertical="1.0471975" width="1200" height="900" rate="5.0"/> -->
     <!-- <xacro:marker_camera link="camera_top_left_link" topic="camera/top/left" fov_horizontal="1.3962634" fov_vertical="1.0471975" width="1200" height="900" rate="5.0"/> -->
     <!-- <xacro:marker_camera link="camera_top_right_link" topic="camera/top/right" fov_horizontal="1.3962634" fov_vertical="1.0471975" width="1200" height="900" rate="5.0"/> -->
-    <xacro:marker_camera link="camera_top_back_link" topic="camera/top/back" fov_horizontal="1.3962634" fov_vertical="1.0471975" width="1200" height="900" rate="5.0"/>
+    <!-- <xacro:marker_camera link="camera_top_back_link" topic="camera/top/back" fov_horizontal="1.3962634" fov_vertical="1.0471975" width="1200" height="900" rate="5.0"/> -->
     <!-- Depth cameras -->
     <xacro:macro name="gemini2" params="name depth_ns color_ns width height rate">
@@ -232,8 +232,8 @@
         </gazebo>
     </xacro:macro>
-    <xacro:gemini2 name="depth_camera_base" depth_ns="/depth/base" color_ns="/camera/base/front" width="640" height="400" rate="10.0"/>
-    <xacro:gemini2 name="depth_camera_top" depth_ns="/depth/top" color_ns="/camera/top/front" width="640" height="400" rate="10.0"/>
-    <!-- Monitor camera -->
-    <xacro:kinematic_link name="monitor_camera" visual="false">
+    <!-- <xacro:gemini2 name="depth_camera_base" depth_ns="/depth/base" color_ns="/camera/base/front" width="640" height="400" rate="10.0"/> -->
+    <!-- <xacro:gemini2 name="depth_camera_top" depth_ns="/depth/top" color_ns="/camera/top/front" width="640" height="400" rate="10.0"/> -->
+    <!-- Monitor camera --> <!-- 4:3 aspect ratio -->
+    <!-- <xacro:kinematic_link name="monitor_camera" visual="false">
         <origin xyz="-1 0 0.7" rpy="0 0.3 0"/>
     </xacro:kinematic_link>
@@ -245,5 +245,5 @@
                 <image>
                     <width>300</width>
-                    <height>225</height> <!-- 4:3 aspect ratio -->
+                    <height>225</height>
                     <format>R8G8B8</format>
                 </image>
@@ -260,5 +260,5 @@
             </plugin>
         </sensor>
-    </gazebo>
+    </gazebo> -->
     <!-- Odometry -->
     <gazebo>
@@ -420,5 +420,5 @@
     </gazebo>
     </xacro:if> -->
-    <gazebo reference="base_link">
+    <!-- <gazebo reference="base_link">
         <material>Gazebo/FlatBlack</material>
         <sensor name="collision_sensor" type="contact">
@@ -434,5 +434,5 @@
             </contact>
         </sensor>
-    </gazebo>
+    </gazebo> -->
     <!-- LED Strips-->
     <xacro:macro name="led_plugin" params="link topic_name">
@@ -445,7 +445,7 @@
         </gazebo>
     </xacro:macro>
-    <xacro:led_plugin link="led0_link" topic_name="gazebo/led0/set_color"/>
+    <!-- <xacro:led_plugin link="led0_link" topic_name="gazebo/led0/set_color"/>
     <xacro:led_plugin link="led1_link" topic_name="gazebo/led1/set_color"/>
     <xacro:led_plugin link="led2_link" topic_name="gazebo/led2/set_color"/>
-    <xacro:led_plugin link="led3_link" topic_name="gazebo/led3/set_color"/>
+    <xacro:led_plugin link="led3_link" topic_name="gazebo/led3/set_color"/> -->
 </robot>

File: workspace/src/controller_launch/models/service_robot/service_robot.xacro (robot description, xacro)
@@ -79,6 +79,6 @@
         </link>
         <joint name="${prefix}_axle_center_joint" type="revolute">
+            <parent link="base_link"/>
             <origin xyz="${-axle_center} ${rear_wheel_separation*reflect} ${base_offset_z + axle_height}" rpy="0 0 0"/>
-            <parent link="base_link"/>
             <child  link="${prefix}_axle_center_link"/>
             <axis xyz="0 1 0" />
@@ -254,9 +254,9 @@
         <origin xyz="${lidar_base_front_x} ${lidar_base_front_y} ${lidar_base_front_z}" rpy="0 0 0"/>
     </joint>
-    <xacro:lidar
+    <!-- <xacro:lidar
         prefix="lidar_base_rear"
         r="${ydlidar_g2_radius}" h="${ydlidar_g2_height}"
         x="${lidar_base_rear_x}" y="${lidar_base_rear_y}" z="${lidar_base_rear_z}"
-        roll="0.0" pitch="0.0" yaw="${lidar_base_rear_yaw}"/>
+        roll="0.0" pitch="0.0" yaw="${lidar_base_rear_yaw}"/> -->
     <!-- Base Depth Camera link -->
     <!-- <xacro:kinematic_link name="depth_camera_base">
@@ -327,7 +327,7 @@
     <xacro:led_strip prefix="led3" filename="file://$(find controller_launch)/led3.stl"/> -->
     <!-- Docking camera -->
-    <xacro:kinematic_link name="camera">
+    <!-- <xacro:kinematic_link name="camera">
         <origin xyz="${cam_pos_x} 0 ${cam_pos_z}" rpy="0 0 ${-pi}" />
-    </xacro:kinematic_link>
+    </xacro:kinematic_link> -->
     <!-- Bumper -->
     <!-- <link name="bumper_link">

Commit message: finalize default nav launch with service robot

File: workspace/src/controller_launch/models/service_robot/plugins.xacro (robot description, xacro)
@@ -59,9 +59,4 @@
         max_angle="${115.0/180*pi}"/> -->
         <!-- [-115°;115°] -->
-    <!-- <joint name="base_joint" type="fixed">
-        <parent>base_footprint</parent>
-        <child>base_link</child>
-        <pose>0.0 0.0 0.010 0 0 0</pose>
-    </joint> -->
     <!-- Diff drive -->
     <gazebo>
@@ -71,6 +66,6 @@
             <odometry_source>1</odometry_source>
             <publish_odom_tf>true</publish_odom_tf>
-            <robot_base_frame>base_link</robot_base_frame>
-            <!-- <robot_base_frame>base_footprint</robot_base_frame> -->
+            <!-- <robot_base_frame>base_link</robot_base_frame> -->
+            <robot_base_frame>base_footprint</robot_base_frame>
             <publish_wheel_tf>false</publish_wheel_tf>
             <publish_wheel_joint_state>true</publish_wheel_joint_state>
@@ -268,5 +263,6 @@
             </ros> -->
             <frame_name>odom</frame_name>
-            <body_name>base_link</body_name>
+            <!-- <body_name>base_link</body_name> -->
+            <body_name>base_footprint</body_name>
             <update_rate>10.0</update_rate>
         </plugin>

File: workspace/src/controller_launch/models/service_robot/service_robot.xacro (robot description, xacro)
@@ -18,4 +18,5 @@
     <xacro:property name="base_front_offset" value="0.02"/>
     <xacro:property name="base_offset_z" value="${base_height/2 + bottom_gap}"/>
+    <link name="base_footprint"/>
     <link name="base_link">
         <xacro:box_inertia
@@ -28,6 +29,11 @@
         </collision>
     </link>
+    <joint name="base_joint" type="fixed">
+        <parent link="base_footprint"/>
+        <child link="base_link"/>
+        <origin xyz="0 0 0" rpy="0 0 0"/>
+    </joint>
     <xacro:property name="base_weight_offset" value="${base_length/8}"/>
-    <link name="battery_link">
+    <!-- <link name="battery_link">
         <xacro:box_inertia
             m="${base_weight}" x="${base_weight_offset*2}" y="${base_width}" z="${base_height}"/>
@@ -37,5 +43,5 @@
         <child  link="battery_link"/>
         <origin xyz="${-base_weight_offset} 0 ${base_offset_z}" rpy="0 0 0"/>
-    </joint>
+    </joint> -->
     <link name="body_link">
         <visual>
